File: ISA_Camac_Interface/ISA_Camac_Interface/ISA_Camac_Interface.sch (KiCad schematic (older format))
At the start: 43 parts

Commit message: path update (in KiCad project)
Parts:
- D1, D2: symbol InterfaceBoard:IC8216 -> ISA_Camac_Interface-rescue:IC8216-InterfaceBoard
- D10: symbol InterfaceBoard:3601 -> ISA_Camac_Interface-rescue:3601-InterfaceBoard
- D11, D12: symbol InterfaceBoard:IC3226 -> ISA_Camac_Interface-rescue:IC3226-InterfaceBoard
- D15: symbol InterfaceBoard:3604 -> ISA_Camac_Interface-rescue:3604-InterfaceBoard
Changed lines of the file:
@@
 $EndDescr
 $Comp
-L InterfaceBoard:3601 D10
+L ISA_Camac_Interface-rescue:3601-InterfaceBoard D10
 U 1 1 5BFFC0EF
 P 5250 1250
@@
 $EndComp
 $Comp
-L InterfaceBoard:3604 D15
+L ISA_Camac_Interface-rescue:3604-InterfaceBoard D15
 U 1 1 5BFFC19E
 P 9400 1400
@@
 $EndComp
 $Comp
-L InterfaceBoard:IC8216 D1
+L ISA_Camac_Interface-rescue:IC8216-InterfaceBoard D1
 U 1 1 5C04B225
 P 3700 3600
@@
 $EndComp
 $Comp
-L InterfaceBoard:IC8216 D2
+L ISA_Camac_Interface-rescue:IC8216-InterfaceBoard D2
 U 1 1 5C04B390
 P 3700 7350
@@
 Z(C2)
 $Comp
-L InterfaceBoard:IC3226 D11
+L ISA_Camac_Interface-rescue:IC3226-InterfaceBoard D11
 U 1 1 5C34E2D9
 P 8950 5300
@@
 $EndComp
 $Comp
-L InterfaceBoard:IC3226 D12
+L ISA_Camac_Interface-rescue:IC3226-InterfaceBoard D12
 U 1 1 5C34E668
 P 8950 9000

Commit message: scheme updated
Parts:
- JP1: value desc -> ADDR1
- JP2: value desc -> ADDR2
Connections:
- net labels added: X2.2(B21)
- net labels removed: X22(B21)
- wire segments 517 -> 522
Other:
- note added: "A11"
- note added: "A2"
- note added: "A22"
- note added: "A23"
- note added: "A24"
- note added: "A25"
- note added: "A26"
- note added: "A27"
- note added: "A28"
- note added: "A29"
- note added: "A3"
- note added: "A30"
- note added: "A31"
- note added: "A4"
- note added: "A5"
- note added: "A6"
- note added: "A7"
- note added: "A8"
- note added: "A9"
- note added: "B2"
- note added: "B28"
- note added: "B3"
- note added: "B4"
- note added: "B5"
- note added: "B6"
- note added: "B7"
- note added: "B8"
- note added: "B9"
- note added: "C2"
- note added: "C3"
- note added: "C4"
- note added: "C5"
- note added: "C6"
- note added: "C7"
- note added: "C8"
- note added: "C9"
- note added: "X1.1\n"
- note added: "X1.2\n"
- note added: "X1.3"
- note added: "X2.1\n"
Changed lines of the file:
@@
 Wire Wire Line
 	2900 3800 3200 3800
-Wire Wire Line
-	2900 3800 1750 3800
 Connection ~ 2900 3800
 Text Label 1750 3800 0    50   ~ 10
 D12
-Wire Wire Line
-	3000 3900 1750 3900
 Connection ~ 3000 3900
 Text Label 1750 3900 0    50   ~ 10
 D14
-Wire Wire Line
-	2950 4000 1750 4000
 Connection ~ 2950 4000
 Text Label 1750 4000 0    50   ~ 10
 D13
-Wire Wire Line
-	3050 4100 1750 4100
 Connection ~ 3050 4100
 Text Label 1750 4100 0    50   ~ 10
@@
 	5750 3750 5750 4450
 Connection ~ 4200 3750
-Wire Wire Line
-	3200 5250 1750 5250
-Wire Wire Line
-	3200 5450 1750 5450
-Wire Wire Line
-	3200 5650 1750 5650
-Wire Wire Line
-	3200 5050 1750 5050
 Text Label 1750 5050 0    50   ~ 10
 D4
@@
 Wire Wire Line
 	3000 9200 3200 9200
-Wire Wire Line
-	3000 9200 1850 9200
 Connection ~ 3000 9200
 Wire Wire Line
@@
 Wire Wire Line
 	2950 9600 3200 9600
-Wire Wire Line
-	2950 9600 1850 9600
 Connection ~ 2950 9600
 Wire Wire Line
@@
 Wire Wire Line
 	2900 9400 3200 9400
-Wire Wire Line
-	2900 9400 1850 9400
 Connection ~ 2900 9400
 Wire Wire Line
@@
 Wire Wire Line
 	2850 9000 3200 9000
-Wire Wire Line
-	2850 9000 1850 9000
 Connection ~ 2850 9000
 Wire Wire Line
@@
 Text Label 1850 9900 0    50   ~ 10
 N(C1)
-Wire Wire Line
-	3200 8900 1850 8900
 Text Label 1850 8900 0    50   ~ 10
 D1
-Wire Wire Line
-	3200 9100 1850 9100
 Text Label 1850 9100 0    50   ~ 10
 D3
-Wire Wire Line
-	3200 9300 1850 9300
 Text Label 1850 9300 0    50   ~ 10
 D2
-Wire Wire Line
-	3200 9500 1850 9500
 Text Label 1850 9500 0    50   ~ 10
 D0
@@
 Text Label 9450 8550 0    50   ~ 0
 D0
-Wire Wire Line
-	8450 9200 7850 9200
-Wire Wire Line
-	8450 9300 7850 9300
-Wire Wire Line
-	8450 9400 7850 9400
-Wire Wire Line
-	8450 9500 7850 9500
 Text Label 7850 9050 0    50   ~ 0
 D(CEL)
@@
 Text Label 8600 7250 0    50   ~ 10
 V(RP)
-Wire Wire Line
-	8000 5500 8450 5500
-Wire Wire Line
-	8000 5600 8450 5600
-Wire Wire Line
-	8000 5700 8450 5700
-Wire Wire Line
-	8000 5800 8450 5800
 Text Label 8000 5800 0    50   ~ 0
 A2(PC_D7)
@@
 Wire Wire Line
 	2350 2100 1950 2100
+Text Label 1950 2100 0    50   ~ 0
+P(WR)
 Text Label 1950 1900 0    50   ~ 0
-P(WR)
-Text Label 1950 2100 0    50   ~ 0
 G(RD)
 Wire Wire Line
-	4750 800  1950 800
-Wire Wire Line
-	4750 900  1950 900
-Wire Wire Line
-	4750 1000 1950 1000
-Wire Wire Line
-	4750 1100 1950 1100
-Wire Wire Line
-	4750 1200 1950 1200
-Wire Wire Line
-	4750 1300 1950 1300
-Wire Wire Line
-	4750 1400 1950 1400
-Wire Wire Line
-	4750 1500 1950 1500
-Wire Wire Line
 	4750 1700 4100 1700
 Wire Wire Line
 	4100 1700 4100 1600
-Wire Wire Line
-	4100 1600 1950 1600
 Text Label 1950 1400 0    50   ~ 0
 A31(PC_A0)
@@
 P 2000 2950
 F 0 "JP2" H 2000 3135 50  0000 C CNN
-F 1 "desc" H 2000 3044 50  0000 C CNN
+F 1 "ADDR2" H 2000 3044 50  0000 C CNN
 F 2 "" H 2000 2950 50  0001 C CNN
 F 3 "~" H 2000 2950 50  0001 C CNN
@@
 P 2000 2700
 F 0 "JP1" H 2000 2885 50  0000 C CNN
-F 1 "desc" H 2000 2794 50  0000 C CNN
+F 1 "ADDR1" H 2000 2794 50  0000 C CNN
 F 2 "" H 2000 2700 50  0001 C CNN
 F 3 "~" H 2000 2700 50  0001 C CNN
@@
 $EndComp
 Wire Wire Line
-	1500 2950 1900 2950
-Wire Wire Line
 	1500 2700 1900 2700
 Text Label 1500 2950 0    50   ~ 0
@@
 Wire Wire Line
 	2350 2500 2350 2400
-Wire Wire Line
-	2350 2400 1500 2400
 Text Label 1500 2400 0    50   ~ 0
 A24(PC_A7)
@@
 Wire Wire Line
 	7350 2000 6600 2000
-Text Label 6600 2000 0    50   ~ 10
-X22(B21)
+Text Label 6600 1850 0    50   ~ 10
+X2.2(B21)
 $Comp
 L Device:R_Small R5
@@
 	14500 6350 14500 6400
 $Comp
-L power:GNDD #PWR?
+L power:GNDD #PWR0101
 U 1 1 5C5B8C40
 P 15000 6500
-F 0 "#PWR?" H 15000 6250 50  0001 C CNN
+F 0 "#PWR0101" H 15000 6250 50  0001 C CNN
 F 1 "GNDD" H 15004 6345 50  0000 C CNN
 F 2 "" H 15000 6500 50  0001 C CNN
@@
 	15000 6500 15000 6350
 $Comp
-L power:GNDD #PWR?
+L power:GNDD #PWR0102
 U 1 1 5C61699B
 P 9850 10200
-F 0 "#PWR?" H 9850 9950 50  0001 C CNN
+F 0 "#PWR0102" H 9850 9950 50  0001 C CNN
 F 1 "GNDD" H 9854 10045 50  0000 C CNN
 F 2 "" H 9850 10200 50  0001 C CNN
@@
 Text Label 12450 9150 0    50   ~ 10
 B25(PC_IRQ3)
+Wire Wire Line
+	950  900  4750 900
+Wire Wire Line
+	950  1000 4750 1000
+Wire Wire Line
+	950  1100 4750 1100
+Wire Wire Line
+	950  1200 4750 1200
+Wire Wire Line
+	950  1300 4750 1300
+Wire Wire Line
+	950  1400 4750 1400
+Wire Wire Line
+	950  1500 4750 1500
+Wire Wire Line
+	950  1600 4100 1600
+Wire Wire Line
+	950  2400 2350 2400
+Wire Wire Line
+	950  800  4750 800
+Wire Wire Line
+	1500 2700 1500 2500
+Wire Wire Line
+	1500 2500 950  2500
+Wire Wire Line
+	1400 2950 1400 2600
+Wire Wire Line
+	1400 2600 950  2600
+Wire Wire Line
+	1400 2950 1900 2950
+Wire Notes Line
+	1050 700  1050 1700
+Text Notes 850  700  0    50   ~ 0
+X1.1\n
+Text Notes 900  800  0    39   ~ 0
+A25
+Text Notes 900  900  0    39   ~ 0
+A26
+Text Notes 900  1000 0    39   ~ 0
+A27
+Text Notes 900  1100 0    39   ~ 0
+A28
+Text Notes 900  1200 0    39   ~ 0
+A29
+Text Notes 900  1300 0    39   ~ 0
+A30
+Text Notes 900  1400 0    39   ~ 0
+A31
+Text Notes 900  1500 0    39   ~ 0
+B28
+Text Notes 900  1600 0    39   ~ 0
+A11
+Wire Wire Line
+	6600 2000 6600 1850
+Connection ~ 6600 2000
+Wire Notes Line
+	1050 2300 1050 2700
+Text Notes 850  2300 0    50   ~ 0
+X1.2\n
+Text Notes 900  2400 0    39   ~ 0
+A24
+Text Notes 900  2500 0    39   ~ 0
+A22
+Text Notes 900  2600 0    39   ~ 0
+A23
+Wire Notes Line
+	1050 3500 1050 10700
+Text Notes 850  3450 0    50   ~ 0
+X2.1\n
+Wire Wire Line
+	950  4100 3050 4100
+Text Notes 900  3800 0    39   ~ 0
+C3
+Text Notes 900  3900 0    39   ~ 0
+C2
+Text Notes 900  4000 0    39   ~ 0
+B3
+Text Notes 900  4100 0    39   ~ 0
+B2
+Text Notes 900  9200 0    39   ~ 0
+B4
+Text Notes 900  9400 0    39   ~ 0
+C4
+Text Notes 900  9000 0    39   ~ 0
+B5
+Wire Wire Line
+	950  9600 2950 9600
+Text Notes 900  9600 0    39   ~ 0
+C5
+Wire Wire Line
+	950  5250 3200 5250
+Wire Wire Line
+	950  5450 3200 5450
+Wire Wire Line
+	950  5650 3200 5650
+Wire Wire Line
+	950  5050 3200 5050
+Text Notes 900  5250 0    39   ~ 0
+B6
+Text Notes 900  5050 0    39   ~ 0
+C7
+Text Notes 900  5450 0    39   ~ 0
+C6
+Text Notes 900  5650 0    39   ~ 0
+B7
+Text Notes 900  8900 0    39   ~ 0
+B9
+Text Notes 900  9100 0    39   ~ 0
+B8
+Text Notes 900  9300 0    39   ~ 0
+C8
+Text Notes 900  9500 0    39   ~ 0
+C9
+Text Notes 7900 5400 0    50   ~ 0
+X1.3
+Wire Notes Line
+	8000 5400 8000 5850
+Wire Wire Line
+	7850 5500 8450 5500
+Wire Wire Line
+	7850 5600 8450 5600
+Wire Wire Line
+	7850 5700 8450 5700
+Wire Wire Line
+	7850 5800 8450 5800
+Text Notes 7800 5500 0    39   ~ 0
+A5
+Text Notes 7800 5600 0    39   ~ 0
+A4
+Text Notes 7800 5700 0    39   ~ 0
+A3
+Text Notes 7800 5800 0    39   ~ 0
+A2
+Wire Notes Line
+	7850 9100 7850 9600
+Wire Wire Line
+	7700 9200 8450 9200
+Wire Wire Line
+	7700 9300 8450 9300
+Wire Wire Line
+	7700 9400 8450 9400
+Wire Wire Line
+	7700 9500 8450 9500
+Text Notes 7650 9200 0    39   ~ 0
+A8
+Text Notes 7650 9300 0    39   ~ 0
+A9
+Text Notes 7650 9400 0    39   ~ 0
+A7
+Text Notes 7650 9500 0    39   ~ 0
+A6
+Text Notes 7650 9100 0    50   ~ 0
+X1.3
+Wire Wire Line
+	950  3800 2900 3800
+Wire Wire Line
+	950  3900 3000 3900
+Wire Wire Line
+	950  4000 2950 4000
+Wire Wire Line
+	950  9200 3000 9200
+Wire Wire Line
+	950  9400 2900 9400
+Wire Wire Line
+	950  9000 2850 9000
+Wire Wire Line
+	950  9100 3200 9100
+Wire Wire Line
+	950  9300 3200 9300
+Wire Wire Line
+	950  9500 3200 9500
+Wire Wire Line
+	950  8900 3200 8900
 Wire Bus Line
 	1750 6300 1750 10350
 Wire Bus Line
+	1650 3650 1650 6300
+Wire Bus Line
 	9650 4750 9650 10500
 Wire Bus Line
-	1650 3650 1650 6300
-Wire Bus Line
 	5000 4500 5000 10350

Commit message: scheme was updated
Parts:
- removed U? (x2): 74LS04, symbol 74xx:74LS04
- gave numbers to parts that had none: 1
Connections:
- net labels added: +5V, CB_A1, CB_A10, CB_A11, CB_A12, CB_A2, CB_A25, CB_A26, CB_A3, CB_A4, CB_A5, CB_A6, CB_A7, CB_A8, CB_A9
- wire segments 522 -> 547
Other:
- note added: "A10"
- note added: "B13"
- note added: "B14"
- note added: "B20"
- note added: "B21"
- note added: "B24"
- note added: "X1.4"
- note added: "X1.5"
- note added: "X2.2"
- note added: "X2.3"
- note added: "X2.4"
Changed lines of the file:
@@
 $EndComp
 $Comp
-L 74xx:74LS04 U?
+L 74xx:74LS04 D18.1
 U 1 1 5C002C60
 P 12550 1250
-F 0 "U?" H 12550 1567 50  0000 C CNN
+F 0 "D18.1" H 12550 1567 50  0000 C CNN
 F 1 "74LS04" H 12550 1476 50  0000 C CNN
 F 2 "" H 12550 1250 50  0001 C CNN
@@
 F 3 "http://www.ti.com/lit/gpn/sn74LS04" H 14000 7800 50  0001 C CNN
 	3    14000 7800
-	1    0    0    -1
-$EndComp
-$Comp
-L 74xx:74LS04 U?
-U 4 1 5C002E87
-P 15600 950
-F 0 "U?" H 15600 1267 50  0000 C CNN
-F 1 "74LS04" H 15600 1176 50  0000 C CNN
-F 2 "" H 15600 950 50  0001 C CNN
-F 3 "http://www.ti.com/lit/gpn/sn74LS04" H 15600 950 50  0001 C CNN
-	4    15600 950
-	1    0    0    -1
-$EndComp
-$Comp
-L 74xx:74LS04 U?
-U 5 1 5C002F5C
-P 15600 1400
-F 0 "U?" H 15600 1717 50  0000 C CNN
-F 1 "74LS04" H 15600 1626 50  0000 C CNN
-F 2 "" H 15600 1400 50  0001 C CNN
-F 3 "http://www.ti.com/lit/gpn/sn74LS04" H 15600 1400 50  0001 C CNN
-	5    15600 1400
 	1    0    0    -1
 $EndComp
@@
 Text Notes 850  3450 0    50   ~ 0
 X2.1\n
-Wire Wire Line
-	950  4100 3050 4100
 Text Notes 900  3800 0    39   ~ 0
 C3
@@
 Text Notes 900  9000 0    39   ~ 0
 B5
-Wire Wire Line
-	950  9600 2950 9600
 Text Notes 900  9600 0    39   ~ 0
 C5
-Wire Wire Line
-	950  5250 3200 5250
-Wire Wire Line
-	950  5450 3200 5450
-Wire Wire Line
-	950  5650 3200 5650
-Wire Wire Line
-	950  5050 3200 5050
 Text Notes 900  5250 0    39   ~ 0
 B6
@@
 X1.3
 Wire Wire Line
+	950  4100 3050 4100
+Wire Wire Line
+	950  9600 2950 9600
+Wire Wire Line
+	950  5250 3200 5250
+Wire Wire Line
+	950  5450 3200 5450
+Wire Wire Line
+	950  5650 3200 5650
+Wire Wire Line
+	950  5050 3200 5050
+Text Notes 13500 1150 0    50   ~ 0
+X1.4
+Text Notes 13550 1200 0    39   ~ 0
+A10
+Text Notes 11300 2600 0    50   ~ 0
+X1.5
+Text Notes 11350 2650 0    39   ~ 0
+B20
+Text Notes 9950 650  0    50   ~ 0
+X2.4
+Text Notes 10000 700  0    39   ~ 0
+B24
+Text Notes 6400 1800 0    50   ~ 0
+X2.2
+Text Notes 6450 1850 0    39   ~ 0
+B21
+Text Notes 10250 3700 0    50   ~ 0
+X1.4
+Text Notes 10300 3750 0    39   ~ 0
+B14
+Text Notes 10250 4450 0    50   ~ 0
+X1.4
+Text Notes 10300 4500 0    39   ~ 0
+B13
+Text Notes 11550 5750 0    50   ~ 0
+X2.3
+Text Notes 11850 5650 0    50   ~ 0
+X1.4
+Text Notes 11800 6700 0    50   ~ 0
+X2.3
+Wire Wire Line
+	15850 2550 15100 2550
+Wire Wire Line
+	15100 2550 15100 2650
+Wire Wire Line
+	15100 2650 15850 2650
+Wire Wire Line
+	15850 2750 15100 2750
+Wire Wire Line
+	15100 2750 15100 2650
+Connection ~ 15100 2650
+Text Label 15700 2550 0    39   ~ 0
+CB_A1
+Text Label 15700 2650 0    39   ~ 0
+CB_A2
+Text Label 15700 2750 0    39   ~ 0
+CB_A3
+Wire Wire Line
+	15850 3100 15100 3100
+Wire Wire Line
+	15100 3100 15100 3200
+Wire Wire Line
+	15100 3200 15850 3200
+$Comp
+L power:GNDD #PWR?
+U 1 1 5C682994
+P 15100 2750
+F 0 "#PWR?" H 15100 2500 50  0001 C CNN
+F 1 "GNDD" H 15104 2595 50  0000 C CNN
+F 2 "" H 15100 2750 50  0001 C CNN
+F 3 "" H 15100 2750 50  0001 C CNN
+	1    15100 2750
+	1    0    0    -1
+$EndComp
+Wire Wire Line
+	15850 3300 15100 3300
+Wire Wire Line
+	15100 3300 15100 3200
+Connection ~ 15100 3200
+Wire Wire Line
+	15850 3400 15100 3400
+Wire Wire Line
+	15100 3400 15100 3300
+Connection ~ 15100 3300
+Wire Wire Line
+	15850 3500 15100 3500
+Wire Wire Line
+	15100 3500 15100 3400
+Connection ~ 15100 3400
+Wire Wire Line
+	15850 3600 15100 3600
+Wire Wire Line
+	15100 3600 15100 3500
+Connection ~ 15100 3500
+Wire Wire Line
+	15100 3700 15100 3600
+Connection ~ 15100 3600
+Wire Wire Line
+	15100 3700 15850 3700
+$Comp
+L power:GNDD #PWR?
+U 1 1 5C9F7E3C
+P 15100 3700
+F 0 "#PWR?" H 15100 3450 50  0001 C CNN
+F 1 "GNDD" H 15104 3545 50  0000 C CNN
+F 2 "" H 15100 3700 50  0001 C CNN
+F 3 "" H 15100 3700 50  0001 C CNN
+	1    15100 3700
+	1    0    0    -1
+$EndComp
+Text Label 15700 3100 0    39   ~ 0
+CB_A4
+Text Label 15700 3200 0    39   ~ 0
+CB_A5
+Text Label 15700 3300 0    39   ~ 0
+CB_A6
+Text Label 15700 3400 0    39   ~ 0
+CB_A7
+Text Label 15700 3500 0    39   ~ 0
+CB_A8
+Text Label 15700 3600 0    39   ~ 0
+CB_A9
+Text Label 15700 3700 0    39   ~ 0
+CB_A10
+Connection ~ 15100 3700
+Wire Wire Line
+	15850 4000 15100 4000
+Wire Wire Line
+	15100 4000 15100 4100
+Wire Wire Line
+	15100 4100 15850 4100
+$Comp
+L power:GNDD #PWR?
+U 1 1 5CBE33B9
+P 15100 4100
+F 0 "#PWR?" H 15100 3850 50  0001 C CNN
+F 1 "GNDD" H 15104 3945 50  0000 C CNN
+F 2 "" H 15100 4100 50  0001 C CNN
+F 3 "" H 15100 4100 50  0001 C CNN
+	1    15100 4100
+	1    0    0    -1
+$EndComp
+Text Label 15700 4000 0    39   ~ 0
+CB_A11
+Text Label 15700 4100 0    39   ~ 0
+CB_A12
+Wire Wire Line
+	15850 4400 15100 4400
+Wire Wire Line
+	15100 4400 15100 4500
+Wire Wire Line
+	15100 4500 15850 4500
+$Comp
+L power:GNDD #PWR?
+U 1 1 5CC358E3
+P 15100 4500
+F 0 "#PWR?" H 15100 4250 50  0001 C CNN
+F 1 "GNDD" H 15104 4345 50  0000 C CNN
+F 2 "" H 15100 4500 50  0001 C CNN
+F 3 "" H 15100 4500 50  0001 C CNN
+	1    15100 4500
+	1    0    0    -1
+$EndComp
+Text Label 15700 4400 0    39   ~ 0
+CB_A25
+Text Label 15700 4500 0    39   ~ 0
+CB_A26
+Wire Wire Line
+	14450 1350 15450 1350
+Wire Wire Line
+	950  8900 3200 8900
+Wire Wire Line
+	950  9100 3200 9100
+Wire Wire Line
+	950  9300 3200 9300
+Wire Wire Line
+	950  9500 3200 9500
+Wire Wire Line
+	950  9400 2900 9400
+Wire Wire Line
+	950  9200 3000 9200
+Wire Wire Line
+	950  9000 2850 9000
+Wire Wire Line
 	950  3800 2900 3800
 Wire Wire Line
@@
 Wire Wire Line
 	950  4000 2950 4000
-Wire Wire Line
-	950  9200 3000 9200
-Wire Wire Line
-	950  9400 2900 9400
-Wire Wire Line
-	950  9000 2850 9000
-Wire Wire Line
-	950  9100 3200 9100
-Wire Wire Line
-	950  9300 3200 9300
-Wire Wire Line
-	950  9500 3200 9500
-Wire Wire Line
-	950  8900 3200 8900
 Wire Bus Line
 	1750 6300 1750 10350
@@
 Wire Bus Line
 	10250 750  10250 3500
+Connection ~ 14450 1350
+Text Label 15450 1350 0    50   ~ 0
++5V
 $EndSCHEMATC

Commit message: sch updated : added uc footprints
Parts:
- added J?: Bus_ISA_8bit, symbol Connector:Bus_ISA_8bit
- D1, D10, D11, D12, D13, D14, D17, D2, D3, D4, D6, D7: footprint (none) -> Package_DIP:DIP-16_W7.62mm_LongPads
- D16, D8: footprint (none) -> Package_DIP:DIP-20_W7.62mm_LongPads
- D18.2, D5.1, D9.3: footprint (none) -> Package_DIP:DIP-14_W7.62mm_LongPads
Other:
- moved on the sheet: C1, D1, D10, D11, D12, D13, D14, D15, D16, D17, D18.1A, D18.2F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

Commit message: scheme updated
Parts:
- X1: renamed from J?; footprint (none) -> InterfaceBoard:ISA_8Bit_Card
Connections:
- net labels added: B14(PC_IOR)
- net labels removed: B14(PC_IQR), L(CEL1)
- wire segments 547 -> 676
Other:
- moved on the sheet: X1

Commit message: scheme changes
Connections:
- wire segments 676 -> 692
Changed lines of the file:
@@
 	9000 8100 8050 8100
 Wire Wire Line
-	8050 6500 8550 6500
+	8050 6500 8350 6500
 Wire Wire Line
 	8550 6500 8550 5500
@@
 Connection ~ 16350 7200
 Wire Wire Line
-	16350 7200 17200 7200
+	16350 7200 16850 7200
 Wire Wire Line
 	18800 3100 18050 3100
@@
 Connection ~ 16350 3500
 Wire Wire Line
-	16350 3500 16350 7200
+	16350 3500 16350 4250
 Wire Wire Line
 	19150 10100 19150 10500
@@
 CB_A26
 Wire Wire Line
-	18800 3100 19800 3100
+	18800 3100 19650 3100
 Connection ~ 18800 3100
-Text Label 19800 3100 0    50   ~ 0
-+5V
 Connection ~ 19450 4500
 Connection ~ 19450 5850
@@
 	10500 900  1550 900
 Wire Wire Line
-	1550 900  1550 2250
-Wire Wire Line
-	1550 2250 2450 2250
-Wire Wire Line
 	10500 5350 15300 5350
 Wire Wire Line
@@
 Wire Wire Line
 	10600 1000 1650 1000
-Wire Wire Line
-	1650 1000 1650 2150
-Wire Wire Line
-	1650 2150 2450 2150
 Wire Wire Line
 	10600 6300 15300 6300
@@
 	1600 3150 2450 3150
 Wire Wire Line
+	16200 10500 17400 10500
+Wire Wire Line
+	2050 1150 2050 4150
+Wire Wire Line
+	2050 4150 2450 4150
+$Comp
+L power:GNDD #PWR?
+U 1 1 63945882
+P 2050 4300
+F 0 "#PWR?" H 2050 4050 50  0001 C CNN
+F 1 "GNDD" H 2054 4145 50  0000 C CNN
+F 2 "" H 2050 4300 50  0001 C CNN
+F 3 "" H 2050 4300 50  0001 C CNN
+	1    2050 4300
+	1    0    0    -1
+$EndComp
+Wire Wire Line
+	2050 4300 2050 4150
+$Comp
+L power:GNDD #PWR?
+U 1 1 639CF9C7
+P 18800 4250
+F 0 "#PWR?" H 18800 4000 50  0001 C CNN
+F 1 "GNDD" H 18804 4095 50  0000 C CNN
+F 2 "" H 18800 4250 50  0001 C CNN
+F 3 "" H 18800 4250 50  0001 C CNN
+	1    18800 4250
+	1    0    0    -1
+$EndComp
+Wire Wire Line
+	18800 4250 18800 4100
+Wire Wire Line
+	14300 3450 14500 3450
+Wire Wire Line
+	14500 3450 14500 4250
+Wire Wire Line
+	14500 4250 16350 4250
+Connection ~ 16350 4250
+Wire Wire Line
+	16350 4250 16350 7200
+$Comp
+L power:+5V #PWR?
+U 1 1 63AE9CD4
+P 19650 3100
+F 0 "#PWR?" H 19650 2950 50  0001 C CNN
+F 1 "+5V" H 19665 3273 50  0000 C CNN
+F 2 "" H 19650 3100 50  0001 C CNN
+F 3 "" H 19650 3100 50  0001 C CNN
+	1    19650 3100
+	1    0    0    -1
+$EndComp
+$Comp
+L power:+5V #PWR?
+U 1 1 63B77DB4
+P 16850 7200
+F 0 "#PWR?" H 16850 7050 50  0001 C CNN
+F 1 "+5V" H 16865 7373 50  0000 C CNN
+F 2 "" H 16850 7200 50  0001 C CNN
+F 3 "" H 16850 7200 50  0001 C CNN
+	1    16850 7200
+	1    0    0    -1
+$EndComp
+Connection ~ 16850 7200
+Wire Wire Line
+	16850 7200 17200 7200
+$Comp
+L power:+5V #PWR?
+U 1 1 63B79620
+P 8350 6500
+F 0 "#PWR?" H 8350 6350 50  0001 C CNN
+F 1 "+5V" H 8365 6673 50  0000 C CNN
+F 2 "" H 8350 6500 50  0001 C CNN
+F 3 "" H 8350 6500 50  0001 C CNN
+	1    8350 6500
+	1    0    0    -1
+$EndComp
+Connection ~ 8350 6500
+Wire Wire Line
+	8350 6500 8550 6500
+Wire Wire Line
+	2050 1150 2450 1150
+Wire Wire Line
+	2450 3950 2200 3950
+Wire Wire Line
+	2200 3950 2200 1450
+Wire Wire Line
+	2200 1350 2450 1350
+Wire Wire Line
+	2200 1450 1850 1450
+Connection ~ 2200 1450
+Wire Wire Line
+	2200 1450 2200 1350
+$Comp
+L power:+5V #PWR?
+U 1 1 63D21EB5
+P 1850 1450
+F 0 "#PWR?" H 1850 1300 50  0001 C CNN
+F 1 "+5V" H 1865 1623 50  0000 C CNN
+F 2 "" H 1850 1450 50  0001 C CNN
+F 3 "" H 1850 1450 50  0001 C CNN
+	1    1850 1450
+	1    0    0    -1
+$EndComp
+Wire Wire Line
+	2450 2350 1650 2350
+Wire Wire Line
+	1650 1000 1650 2350
+Wire Wire Line
+	2450 2450 1550 2450
+Wire Wire Line
+	1550 900  1550 2450
+Wire Wire Line
 	5300 10650 7550 10650
 Wire Wire Line
@@
 Wire Wire Line
 	5300 5750 7300 5750
-Wire Wire Line
-	16200 10500 17400 10500
 Wire Bus Line
 	6100 8050 6100 12100
